File: KiCad/GR_KS0835F_SLIC_Breakout.kicad_pcb (KiCad board)
At the start: 2 copper layers, 71.7 x 27.7 mm, 25 parts, among them J1 RJ, J2 Conn_01x10, U1 KS0835F

Commit message: Add files via upload
Parts:
- D6: footprint Diode_THT:D_DO-41_SOD81_P10.16mm_Horizontal -> Diode_THT:D_DO-15_P12.70mm_Horizontal
- moved D6 1.05 mm to (142.6, 125.6)
Routing:
- net /F_R: track 36.5 -> 37.4 mm
- net /RM: track 39.8 -> 40.6 mm
